File: Schematic/Mixer.kicad_sch (KiCad schematic)
At the start: 83 parts, among them U1001 TL074, U1002 TL074, U1003 TL074, U1004 TL074, U1005 TL074

Commit message: cleansing fire
Connections:
- net +12V: now also U1005.4 (V+); no longer U1005.11 (V-)
- net -12V: now also U1005.11 (V-); no longer U1005.4 (V+)
Changed lines of the file:
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@@
     )
   )
-  (symbol (lib_id "Amplifier_Operational:TL074") (at 38.1 205.74 0) (mirror x) (unit 5)
+  (symbol (lib_id "Amplifier_Operational:TL074") (at 33.02 205.74 0) (mirror y) (unit 5)
     (in_bom yes) (on_board yes) (dnp no) (fields_autoplaced)
-    (property "Reference" "U1005" (at 34.9251 204.5279 0)
+    (property "Reference" "U1005" (at 36.83 204.47 0)
       (effects (font (size 1.27 1.27)) (justify right))
     )
-    (property "Value" "TL074" (at 34.9251 206.9521 0)
+    (property "Value" "TL074" (at 36.83 207.01 0)
       (effects (font (size 1.27 1.27)) (justify right))
     )
-    (property "Footprint" "Package_DIP:DIP-14_W7.62mm" (at 36.83 208.28 0)
+    (property "Footprint" "Package_DIP:DIP-14_W7.62mm" (at 34.29 203.2 0)
       (effects (font (size 1.27 1.27)) hide)
     )
-    (property "Datasheet" "http://www.ti.com/lit/ds/symlink/tl071.pdf" (at 39.37 210.82 0)
+    (property "Datasheet" "http://www.ti.com/lit/ds/symlink/tl071.pdf" (at 31.75 200.66 0)
       (effects (font (size 1.27 1.27)) hide)
     )
