File: Schematic/Output.kicad_sch (KiCad schematic)
At the start: 28 parts, among them J901 M_IN, J902 KEYPAD, J904 POWER, J905 TRIG, J906 READER, J907 ENC1, J908 ENC2, J909 DISP1, J910 DISP2, J911 M_OUT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

Commit message: cleansing fire
Parts:
- removed J912: AUX_IN, TerminalBlock_Phoenix:TerminalBlock_Phoenix_MKDS-1,5-2_1x02_P5.00mm_Horizontal, symbol Connector:Screw_Terminal_01x02
Other:
- note removed: "Screw terminal for connecting the I2S amp output back to the mixer"
Changed lines of the file:
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@@
-    (stroke (width 0) (type default))
-  )
-  (wire (pts (xy 218.44 29.21) (xy 223.52 29.21))
     (stroke (width 0) (type default))
   )
@@
   )
   (wire (pts (xy 64.77 95.25) (xy 68.58 95.25))
-    (stroke (width 0) (type default))
-  )
-  (wire (pts (xy 223.52 31.75) (xy 223.52 36.83))
     (stroke (width 0) (type default))
   )
@@
   )
   (text "Input MIDI DIN jack" (at 48.26 22.86 0)
-    (effects (font (size 1.27 1.27)) (justify left bottom))
-  )
-  (text "Screw terminal for connecting the I2S amp output back to the mixer"
-    (at 205.74 25.4 0)
     (effects (font (size 1.27 1.27)) (justify left bottom))
   )
@@
     )
   )
-  (global_label "Aux" (shape input) (at 218.44 29.21 180) (fields_autoplaced)
-    (effects (font (size 1.27 1.27)) (justify right))
-    (property "Intersheetrefs" "${INTERSHEET_REFS}" (at 212.8433 29.21 0)
-      (effects (font (size 1.27 1.27)) (justify right) hide)
-    )
-  )
   (global_label "Kick2Out" (shape input) (at 64.77 82.55 180) (fields_autoplaced)
     (effects (font (size 1.27 1.27)) (justify right))
@@
         (path "/36804e49-266f-4323-9d1a-a2cb3256aa72/00000000-0000-0000-0000-0000650ea811"
           (reference "C908") (unit 1)
-        )
-      )
-    )
-  )
-  (symbol (lib_id "Connector:Screw_Terminal_01x02") (at 228.6 29.21 0) (unit 1)
-    (in_bom yes) (on_board yes) (dnp no) (fields_autoplaced)
-    (property "Reference" "J912" (at 231.14 29.21 0)
-      (effects (font (size 1.27 1.27)) (justify left))
-    )
-    (property "Value" "AUX_IN" (at 231.14 31.75 0)
-      (effects (font (size 1.27 1.27)) (justify left))
-    )
-    (property "Footprint" "TerminalBlock_Phoenix:TerminalBlock_Phoenix_MKDS-1,5-2_1x02_P5.00mm_Horizontal" (at 228.6 29.21 0)
-      (effects (font (size 1.27 1.27)) hide)
-    )
-    (property "Datasheet" "~" (at 228.6 29.21 0)
-      (effects (font (size 1.27 1.27)) hide)
-    )
-    (pin "1")
-    (pin "2")
-    (instances
-      (project "ESP808"
-        (path "/36804e49-266f-4323-9d1a-a2cb3256aa72/00000000-0000-0000-0000-0000650ea811"
-          (reference "J912") (unit 1)
         )
       )
@@
         )
       )
-    )
-  )
-  (symbol (lib_id "PCM_4ms_Power-symbol:GND") (at 223.52 36.83 0) (unit 1)
-    (in_bom yes) (on_board yes) (dnp no) (fields_autoplaced)
-    (property "Reference" "#PWR0936" (at 223.52 43.18 0)
-      (effects (font (size 1.27 1.27)) hide)
-    )
-    (property "Value" "GND" (at 223.52 41.91 0)
-      (effects (font (size 1.27 1.27)))
-    )
-    (property "Footprint" "" (at 223.52 36.83 0)
-      (effects (font (size 1.27 1.27)) hide)
-    )
-    (property "Datasheet" "" (at 223.52 36.83 0)
-      (effects (font (size 1.27 1.27)) hide)
-    )
-    (pin "1")
-    (instances
-      (project "ESP808"
-        (path "/36804e49-266f-4323-9d1a-a2cb3256aa72/00000000-0000-0000-0000-0000650ea811"
-          (reference "#PWR0936") (unit 1)
-        )
-      )
